File: Arduino Sequencer.kicad_sch (KiCad schematic)
At the start: 16 parts, among them J1 AudioJack2, J2 AudioJack2, J3 AudioJack2, J4 AudioJack2, SW1 Selector, U1 MCP4728

Commit message: include new modifiers
Parts:
- added C1, C3: 1uF, Capacitor_THT:CP_Radial_D6.3mm_P2.50mm, symbol Device:C
- added C2: 10uF, Capacitor_THT:CP_Radial_D6.3mm_P2.50mm, symbol Device:C
- added D5, D6: 1N4148, Diode_THT:D_DO-27_P5.08mm_Vertical_AnodeUp, symbol Device:D
- added J5: Eurorack Power, Connector_PinHeader_1.00mm:PinHeader_2x05_P1.00mm_Vertical, symbol Connector_Generic:Conn_02x05_Top_Bottom
- added U3: L7805, symbol Regulator_Linear:L7805
- D1, D2, D3, D4: footprint (none) -> LED_THT:LED_D4.0mm
- J1, J2, J3, J4: footprint (none) -> Connector_Audio:Jack_3.5mm_QingPu_WQP-PJ398SM_Vertical_CircularHoles
- R1, R2, R3, R4: value R_Small -> 220; footprint (none) -> Resistor_THT:R_Box_L13.0mm_W4.0mm_P9.00mm
- SW1: footprint (none) -> Rotary_Encoder:RotaryEncoder_Alps_EC11E-Switch_Vertical_H20mm
Connections:
- net +5V: no longer A1.27 (+5V)
- net GND: now also A1.6 (D3), SW1.A, C1.2, C2.1, C3.1, J5.2 (Pin_2), J5.3 (Pin_3), J5.4 (Pin_4), J5.7 (Pin_7), J5.8 (Pin_8), J5.9 (Pin_9), U3.2 (GND)
- new net: C1.1, D6.1 (K), U3.1 (IN)
- new net: A1.27 (+5V), C2.2, C3.2, U3.3 (OUT)
- new net: D6.2 (A), J5.1 (Pin_1), J5.6 (Pin_6)
- new net: D5.2 (A), J5.10 (Pin_10), J5.5 (Pin_5)
- new net -12V: D5.1 (K)
Other:
- moved on the sheet: A1, D1, D2, D3, D4, J1, J2, J3, J4, R1, R2, R3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
